Commit message: tractor sim

File: gazebo_tractor_sim_pkg/urdf/my_robot.xacro (robot description, xacro)
@@ -36,5 +36,5 @@
       <origin xyz="0 0 0" rpy=" 0 1.5707 1.5707"/>
       <geometry>
-        <cylinder radius="0.2" length="0.09"/>
+        <cylinder radius="0.2" length="0.1"/>
       </geometry>
     </collision>
@@ -51,5 +51,5 @@
       <origin xyz="0 0 0" rpy=" 0 1.5707 1.5707"/>
       <geometry>
-        <cylinder radius="0.2" length="0.09"/>
+        <cylinder radius="0.2" length="0.1"/>
       </geometry>
     </visual>
@@ -59,5 +59,5 @@
       <origin xyz="0 0 0" rpy=" 0 1.5707 1.5707"/>
       <geometry>
-        <cylinder radius="0.2" length="0.09"/>
+        <cylinder radius="0.2" length="0.1"/>
       </geometry>
     </collision>
@@ -74,5 +74,5 @@
       <origin xyz="0 0 0" rpy=" 0 1.5707 1.5707"/>
       <geometry>
-        <cylinder radius="0.2" length="0.09"/>
+        <cylinder radius="0.2" length="0.1"/>
       </geometry>
     </visual>
@@ -82,5 +82,5 @@
       <origin xyz="0 0 0" rpy=" 0 1.5707 1.5707"/>
       <geometry>
-        <cylinder radius="0.2" length="0.09"/>
+        <cylinder radius="0.2" length="0.1"/>
       </geometry>
     </collision>
@@ -97,5 +97,5 @@
       <origin xyz="0 0 0" rpy=" 0 1.5707 1.5707"/>
       <geometry>
-        <cylinder radius="0.2" length="0.09"/>
+        <cylinder radius="0.2" length="0.1"/>
       </geometry>
     </visual>
@@ -105,5 +105,5 @@
       <origin xyz="0 0 0" rpy=" 0 1.5707 1.5707"/>
       <geometry>
-        <cylinder radius="0.2" length="0.09"/>
+        <cylinder radius="0.2" length="0.1"/>
       </geometry>
     </collision>
@@ -120,5 +120,5 @@
       <origin xyz="0 0 0" rpy=" 0 1.5707 1.5707"/>
       <geometry>
-        <cylinder radius="0.2" length="0.09"/>
+        <cylinder radius="0.2" length="0.1"/>
       </geometry>
     </visual>
